File: pcb/v1.1/DeskHop_Rev1.kicad_pcb (KiCad board)
At the start: 2 copper layers, 66.9 x 74.5 mm, 20 parts, among them J1 Keyboard In, J2 Debug2, J3 Debug1, J4 Mouse In, U1 Pico Primary, U2 Pico Secondary, U3 TPD4E1U06DBVR, U4 ADuM1201BR, U5 TPD4E1U06DBVR

Commit message: update smd r/c to 1206 size
Parts:
- C1, C2, C3, C4: footprint Capacitor_SMD:C_0805_2012Metric -> Capacitor_SMD:C_1206_3216Metric_Pad1.33x1.80mm_HandSolder
- R1, R2, R3, R4: footprint Resistor_SMD:R_0805_2012Metric -> Resistor_SMD:R_1206_3216Metric_Pad1.30x1.75mm_HandSolder
